File: SSTCGV.kicad_pcb (KiCad board)
At the start: 2 copper layers, 46 parts, among them IC1 ATTINY13-20PU, J1-1 INPUT 1, J1-2 INPUT 2, J2 COILS, J3 POWER, J4 OPT, Q1 IRLZ44N, Q2 IRLZ44N, Q3 IRLZ44N, SW1 SW_Push_DPDT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

Commit message: woking on pcb
Parts:
- removed J1-1: INPUT 1, Connector_PinSocket_2.54mm:PinSocket_1x04_P2.54mm_Vertical
- removed J1-2: INPUT 2, Connector_PinSocket_2.54mm:PinSocket_1x04_P2.54mm_Vertical
- D2: footprint LED_THT:LED_D5.0mm-3_Horizontal_O3.81mm_Z3.0mm -> LED_THT:LED_D5.0mm-3
- R1: footprint Resistor_THT:R_Axial_DIN0411_L9.9mm_D3.6mm_P15.24mm_Horizontal -> Resistor_THT:R_Axial_DIN0309_L9.0mm_D3.2mm_P5.08mm_Vertical
- R2, R3, R4, R5, R6, R8, R9, RO1, RO2: footprint Resistor_THT:R_Axial_DIN0411_L9.9mm_D3.6mm_P15.24mm_Horizontal -> Resistor_THT:R_Axial_DIN0411_L9.9mm_D3.6mm_P7.62mm_Vertical
- moved C9 140.9 mm to (231.2, 127.0)
- moved C10 127.2 mm to (231.1, 121.9)
- moved J2 127.1 mm to (83.8, 160.0), turned to -90 degrees
- moved IC1 117.1 mm to (86.4, 139.7)
- moved C8 108.1 mm to (231.1, 116.8)
- moved R6 102.5 mm to (170.2, 132.1), turned to -90 degrees
- moved J3 98.7 mm to (48.3, 116.8)
- moved L1 94.1 mm to (236.2, 106.7), turned to -90 degrees
- moved D8 92.2 mm to (210.8, 137.2)
- moved R5 88.1 mm to (142.2, 142.2)
- moved RV2 85.7 mm to (58.4, 160.0)
- moved D5 81.0 mm to (210.8, 127.0)
- moved D3 80.2 mm to (193.0, 111.8)
- moved D4 78.9 mm to (210.8, 106.7)
- moved R3 74.7 mm to (142.2, 132.1)
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Connections:
- C3 pad 1: Net-(IC1-Pad3) -> Net-(C3-Pad1)
- CO1 pad 2: Net-(CO1-Pad2) -> GND
- IC1 pad 3: Net-(IC1-Pad3) -> Net-(C3-Pad1)
- IC1 pad 5: Net-(R3-Pad1) -> Net-(CO1-Pad1)
- R2 pad 1: Net-(IC1-Pad3) -> Net-(C3-Pad1)
- R3 pad 1: Net-(R3-Pad1) -> Net-(CO1-Pad1)
- RO2 pad 2: Net-(CO1-Pad2) -> GND
- RV2 pad 1: Net-(CO1-Pad2) -> GND
- RV2 pad 3: Net-(U1-Pad4) -> +5V
- SW1 pad 2: Net-(CO1-Pad2) -> GND
- SW1 pad 5: Net-(J1-2-Pad3) -> Net-(C3-Pad1)
- U1 pad 4: Net-(U1-Pad4) -> +5V
